File: ESP32_Plotter_Controller.sch (KiCad schematic (older format))
At the start: 34 parts, among them J1 ARM JTAG 10pin, J10 Pen Lift, J11 Vselect, J12 X Motor, J13 Y Motor, J14 Neo Pixel LEDs, J15 Pen Direction, J16 Aux Port (I2C), J2 Power, J3 5V Aux, J4 Vin Aux, J5 Limit Switches, J6 Aux Port (SPI), J7 X Limit, J8 Micro_SD_Card_TF-01A, J9 Y Limit, U1 ESP-DEVKITC, U2 TMC2130, U3 TMC2130, U4 XL1509

Commit message: Update repo links
Other:
- note added: "ESP32 Plotter Controller\nDesign by Mark Benson\ngithub.com/theworkisthework/ESP32_Plotter_Controller\nBased on Bart Drings ESP32 Pen Plotter Controller\nhttps://github.com/bdring/Grbl_ESP32_TMC2130_Plotter_Controller"
- note removed: "ESP32 Plotter Controller\nDesign by Mark Benson github.com/markjb/ESP32_Plotter_Controller\nBased on Bart Drings ESP32 Pen Plotter Controller\nhttps://github.com/bdring/Grbl_ESP32_TMC2130_Plotter_Controller"
Changed lines of the file:
@@
 $EndComp
 Text Notes 15000 12575 0    79   ~ 0
-ESP32 Plotter Controller\nDesign by Mark Benson github.com/markjb/ESP32_Plotter_Controller\nBased on Bart Drings ESP32 Pen Plotter Controller\nhttps://github.com/bdring/Grbl_ESP32_TMC2130_Plotter_Controller
+ESP32 Plotter Controller\nDesign by Mark Benson\ngithub.com/theworkisthework/ESP32_Plotter_Controller\nBased on Bart Drings ESP32 Pen Plotter Controller\nhttps://github.com/bdring/Grbl_ESP32_TMC2130_Plotter_Controller
 Text Label 6530 5300 2    50   ~ 0
 CS_AUX
