File: ESP32_Plotter_Controller_revA.kicad_pcb (KiCad board)
At the start: 2 copper layers, 99.1 x 55.4 mm, 40 parts, among them J1 ARM JTAG 10pin, J10 Pen Lift, J11 Vselect, J12 X Motor, J13 Y Motor, J14 Neo Pixel LEDs, J15 Pen Direction, J16 Aux Port (I2C), J2 Power, J3 5V Aux, J4 Vin Aux, J5 Limit Switches, J6 Aux Port (SPI), J7 X Limit, J8 Micro_SD_Card_TF-01A, J9 Y Limit, U1 ESP-DEVKITC, U2 TMC2130, U3 TMC2130, U4 XL1509

Commit message: Update repo links
Other:
- board text added: "github.com/theworkisthework/ESP32_Plotter_Controller"
- board text removed: "github.com/markjb/ESP32_Plotter_Controller"
